File: kicad/automato.kicad_pcb (KiCad board)
At the start: 4 copper layers, 106 x 64 mm, 84 parts, among them J1 USB_C_Receptacle, J10 QWIIC 0, J12 STEMMA 0, J2 LiPo, J4 Screw_Terminal_01x14, J5 USB_C_Receptacle, J6 Conn_Coaxial, J7 1-WIRE, J8 Micro_SD_Card_Det, J9 UART2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

Commit message: update
Parts:
- removed REF** (x4): MountingHole_3.2mm_M3_DIN965_Pad_TopBottom, MountingHole:MountingHole_3.2mm_M3_DIN965_Pad_TopBottom
- renumbered U8 to U4
Connections:
- JP1 pad 3: IO15 -> IO16
- JP2 pad 3: IO16 -> IO17
- Q6 pad 1: IO15 -> IO16
- Q6 pad 4: IO16 -> IO17
- U4 pad 14: CS_RELAY -> CS_SD
- U4 pad 17: IO13 -> CS_RELAY
- U4 pad 30: SPI_CLK -> IO17
- U4 pad 31: CS_SD -> IRQ_LORA
- U4 pad 32: SPI_MISO -> SPI_CLK
- U4 pad 33: I2C_SDA -> SPI_MISO
- U4 pad 35: I2C_SCL -> I2C_SDA
- U4 pad 38: SPI_MOSI -> I2C_SCL
- U4 pad 39: RST_EINK -> SPI_MOSI
- U4 pad 9: IRQ_LORA -> RST_EINK
Changed lines of the file:
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@@
     (tracks 1064)
     (zones 0)
-    (modules 84)
-    (nets 112)
+    (modules 80)
+    (nets 113)
   )
   (page A4)
@@
   (net 110 "Net-(J12-Pad3)")
   (net 111 "Net-(J12-Pad2)")
+  (net 112 IO17)
   (net_class Default "This is the default net class."
     (clearance 0.2)
@@
     (add_net IO15)
     (add_net IO16)
+    (add_net IO17)
     (add_net IRQ_LORA)
     (add_net "Net-(C13-Pad1)")
@@
     (add_net VIN)
   )
-  (module MountingHole:MountingHole_3.2mm_M3_DIN965_Pad_TopBottom (layer F.Cu)
-    (at 83.1 117.9)
-    (descr "Mounting Hole 3.2mm, M3, DIN965")
-    (tags "mounting hole 3.2mm m3 din965")
-    (attr virtual)
-    (fp_text reference REF** (at 0 -3.8) (layer F.SilkS)
-      (effects (font (size 1 1) (thickness 0.15)))
-    )
-    (fp_text value MountingHole_3.2mm_M3_DIN965_Pad_TopBottom (at 0 3.8) (layer F.Fab)
-      (effects (font (size 1 1) (thickness 0.15)))
-    )
-    (fp_text user %R (at 0.3 0) (layer F.Fab)
-      (effects (font (size 1 1) (thickness 0.15)))
-    )
-    (fp_circle (center 0 0) (end 2.8 0) (layer Cmts.User) (width 0.15))
-    (fp_circle (center 0 0) (end 3.05 0) (layer F.CrtYd) (width 0.05))
-    (pad 1 connect circle (at 0 0) (size 5.6 5.6) (layers B.Cu B.Mask))
-    (pad 1 connect circle (at 0 0) (size 5.6 5.6) (layers F.Cu F.Mask))
-    (pad 1 thru_hole circle (at 0 0) (size 3.6 3.6) (drill 3.2) (layers *.Cu *.Mask))
-  )
-  (module MountingHole:MountingHole_3.2mm_M3_DIN965_Pad_TopBottom (layer F.Cu)
-    (at 182.9 117.9)
-    (descr "Mounting Hole 3.2mm, M3, DIN965")
-    (tags "mounting hole 3.2mm m3 din965")
-    (attr virtual)
-    (fp_text reference REF** (at 0 -3.8) (layer F.SilkS)
-      (effects (font (size 1 1) (thickness 0.15)))
-    )
-    (fp_text value MountingHole_3.2mm_M3_DIN965_Pad_TopBottom (at 0 3.8) (layer F.Fab)
-      (effects (font (size 1 1) (thickness 0.15)))
-    )
-    (fp_text user %R (at 0.3 0) (layer F.Fab)
-      (effects (font (size 1 1) (thickness 0.15)))
-    )
-    (fp_circle (center 0 0) (end 2.8 0) (layer Cmts.User) (width 0.15))
-    (fp_circle (center 0 0) (end 3.05 0) (layer F.CrtYd) (width 0.05))
-    (pad 1 connect circle (at 0 0) (size 5.6 5.6) (layers B.Cu B.Mask))
-    (pad 1 connect circle (at 0 0) (size 5.6 5.6) (layers F.Cu F.Mask))
-    (pad 1 thru_hole circle (at 0 0) (size 3.6 3.6) (drill 3.2) (layers *.Cu *.Mask))
-  )
-  (module MountingHole:MountingHole_3.2mm_M3_DIN965_Pad_TopBottom (layer F.Cu)
-    (at 182.9 60.1)
-    (descr "Mounting Hole 3.2mm, M3, DIN965")
-    (tags "mounting hole 3.2mm m3 din965")
-    (attr virtual)
-    (fp_text reference REF** (at 0 -3.8) (layer F.SilkS)
-      (effects (font (size 1 1) (thickness 0.15)))
-    )
-    (fp_text value MountingHole_3.2mm_M3_DIN965_Pad_TopBottom (at 0 3.8) (layer F.Fab)
-      (effects (font (size 1 1) (thickness 0.15)))
-    )
-    (fp_text user %R (at 0.3 0) (layer F.Fab)
-      (effects (font (size 1 1) (thickness 0.15)))
-    )
-    (fp_circle (center 0 0) (end 2.8 0) (layer Cmts.User) (width 0.15))
-    (fp_circle (center 0 0) (end 3.05 0) (layer F.CrtYd) (width 0.05))
-    (pad 1 connect circle (at 0 0) (size 5.6 5.6) (layers B.Cu B.Mask))
-    (pad 1 connect circle (at 0 0) (size 5.6 5.6) (layers F.Cu F.Mask))
-    (pad 1 thru_hole circle (at 0 0) (size 3.6 3.6) (drill 3.2) (layers *.Cu *.Mask))
-  )
-  (module MountingHole:MountingHole_3.2mm_M3_DIN965_Pad_TopBottom (layer F.Cu)
-    (at 83.2 60.1)
-    (descr "Mounting Hole 3.2mm, M3, DIN965")
-    (tags "mounting hole 3.2mm m3 din965")
-    (attr virtual)
-    (fp_text reference REF** (at 0 -3.8) (layer F.SilkS)
-      (effects (font (size 1 1) (thickness 0.15)))
-    )
-    (fp_text value MountingHole_3.2mm_M3_DIN965_Pad_TopBottom (at 0 3.8) (layer F.Fab)
-      (effects (font (size 1 1) (thickness 0.15)))
-    )
-    (fp_text user %R (at 0.3 0) (layer F.Fab)
-      (effects (font (size 1 1) (thickness 0.15)))
-    )
-    (fp_circle (center 0 0) (end 2.8 0) (layer Cmts.User) (width 0.15))
-    (fp_circle (center 0 0) (end 3.05 0) (layer F.CrtYd) (width 0.05))
-    (pad 1 connect circle (at 0 0) (size 5.6 5.6) (layers B.Cu B.Mask))
-    (pad 1 connect circle (at 0 0) (size 5.6 5.6) (layers F.Cu F.Mask))
-    (pad 1 thru_hole circle (at 0 0) (size 3.6 3.6) (drill 3.2) (layers *.Cu *.Mask))
-  )
   (module automato-sensor:ESP32-WROOM-DA (layer F.Cu)
     (at 149 76.25)
-    (fp_text reference U8 (at 2.2 1.9) (layer F.SilkS)
+    (fp_text reference U4 (at 2.2 1.9) (layer F.SilkS)
       (effects (font (size 1 1) (thickness 0.15)))
     )
@@
       (net 1 GND))
     (pad 39 smd rect (at 17.75 -16.74) (size 1.5 0.9) (layers F.Cu F.Paste F.Mask)
-      (net 94 RST_EINK))
+      (net 29 SPI_MOSI))
     (pad 38 smd rect (at 17.75 -15.47) (size 1.5 0.9) (layers F.Cu F.Paste F.Mask)
-      (net 29 SPI_MOSI))
+      (net 27 I2C_SCL))
     (pad 37 smd rect (at 17.75 -14.2) (size 1.5 0.9) (layers F.Cu F.Paste F.Mask)
       (net 25 TX))
@@
       (net 24 RX))
     (pad 35 smd rect (at 17.75 -11.66) (size 1.5 0.9) (layers F.Cu F.Paste F.Mask)
-      (net 27 I2C_SCL))
+      (net 26 I2C_SDA))
     (pad 34 smd rect (at 17.75 -10.39) (size 1.5 0.9) (layers F.Cu F.Paste F.Mask))
     (pad 33 smd rect (at 17.75 -9.12) (size 1.5 0.9) (layers F.Cu F.Paste F.Mask)
-      (net 26 I2C_SDA))
+      (net 30 SPI_MISO))
     (pad 32 smd rect (at 17.75 -7.85) (size 1.5 0.9) (layers F.Cu F.Paste F.Mask)
-      (net 30 SPI_MISO))
+      (net 31 SPI_CLK))
     (pad 31 smd rect (at 17.75 -6.58) (size 1.5 0.9) (layers F.Cu F.Paste F.Mask)
-      (net 28 CS_SD))
+      (net 41 IRQ_LORA))
     (pad 30 smd rect (at 17.75 -5.31) (size 1.5 0.9) (layers F.Cu F.Paste F.Mask)
-      (net 31 SPI_CLK))
+      (net 112 IO17))
     (pad 29 smd rect (at 17.75 -4.04) (size 1.5 0.9) (layers F.Cu F.Paste F.Mask)
       (net 96 IO16))
@@
       (net 1 GND))
     (pad 14 smd rect (at 0.25 -1.5) (size 1.5 0.9) (layers F.Cu F.Paste F.Mask)
-      (net 91 CS_RELAY))
+      (net 28 CS_SD))
     (pad 13 smd rect (at 0.25 -2.77) (size 1.5 0.9) (layers F.Cu F.Paste F.Mask)
       (net 99 IO14))
@@
     (pad 10 smd rect (at 0.25 -6.58) (size 1.5 0.9) (layers F.Cu F.Paste F.Mask))
     (pad 9 smd rect (at 0.25 -7.85) (size 1.5 0.9) (layers F.Cu F.Paste F.Mask)
-      (net 41 IRQ_LORA))
+      (net 94 RST_EINK))
     (pad 8 smd rect (at 0.25 -9.12) (size 1.5 0.9) (layers F.Cu F.Paste F.Mask)
       (net 95 BUSY_EINK))
@@
     (pad 18 smd rect (at 5.825 -0.25 90) (size 1.5 0.9) (layers F.Cu F.Paste F.Mask))
     (pad 17 smd rect (at 4.555 -0.25 90) (size 1.5 0.9) (layers F.Cu F.Paste F.Mask)
-      (net 98 IO13))
+      (net 91 CS_RELAY))
     (pad 16 smd rect (at 3.285 -0.25 90) (size 1.5 0.9) (layers F.Cu F.Paste F.Mask)
       (net 1 GND))
@@
       (net 103 "Net-(J9-Pad4)"))
     (pad 4 smd rect (at 1.1 0.95 90) (size 1.06 0.65) (layers F.Cu F.Paste F.Mask)
-      (net 96 IO16))
+      (net 112 IO17))
     (pad 3 smd rect (at -1.1 0.95 90) (size 1.06 0.65) (layers F.Cu F.Paste F.Mask)
       (net 104 "Net-(J9-Pad3)"))
@@
       (net 101 +3V3))
     (pad 1 smd rect (at -1.1 -0.95 90) (size 1.06 0.65) (layers F.Cu F.Paste F.Mask)
-      (net 97 IO15))
+      (net 96 IO16))
     (model ${KISYS3DMOD}/Package_TO_SOT_SMD.3dshapes/SOT-23-6.wrl
       (at (xyz 0 0 0))
@@
     (fp_arc (start -1.35 -0.3) (end -1.35 -1) (angle -90) (layer F.SilkS) (width 0.12))
     (pad 3 smd custom (at 1.3 0 180) (size 1 0.5) (layers F.Cu F.Mask)
-      (net 96 IO16) (zone_connect 2)
+      (net 112 IO17) (zone_connect 2)
       (options (clearance outline) (anchor rect))
       (primitives
@@
     (fp_arc (start -1.35 -0.3) (end -1.35 -1) (angle -90) (layer F.SilkS) (width 0.12))
     (pad 3 smd custom (at 1.3 0 180) (size 1 0.5) (layers F.Cu F.Mask)
-      (net 97 IO15) (zone_connect 2)
+      (net 96 IO16) (zone_connect 2)
       (options (clearance outline) (anchor rect))
       (primitives
